Commit message: [modify] descriptionファイルを修正
見やすくなるように、細かいところを修正

File: model_description/urdf/sensor/camera.gazebo.xacro (robot description, xacro)
@@ -1,13 +1,12 @@
 <?xml version="1.0"?>
 <robot xmlns:xacro="http://ros.org/wiki/xacro">
-  <xacro:include filename="$(find model_description)/urdf/common.xacro" />
-  <xacro:include filename="$[find model_description]/urdf/materials.xacro"/>
-  <xacro:macro name="gscam_gazebo" parames="link_name">
-	<gazebo reference="${link_name}">
+  <xacro:include filename="$(find model_description)/urdf/common.xacro"/>
+  <xacro:macro name="gscam_gazebo" params="name">
+	<gazebo reference="${name}">
 	  <material>Gazebo/Black</material>
-	  <sensor type="camera" name="gscam">
+	  <sensor type="camera" name="gscam1">
 		<update_rate>60.0</update_rate>
-		<camera name="gscam">
-          <horizontal_fov>1.570796</horizontal_fov>
+		<camera name="head">
+          <horizontal_fov>${M_PI/2}</horizontal_fov>
           <image>
 			<width>744</width>
@@ -25,5 +24,5 @@
           </noise>
 		</camera>
-		<plugin name="camera_controller" filename="libgazebo_ros_camera.so">
+		<plugin name="${name}_controller" filename="libgazebo_ros_camera.so">
           <alwaysOn>true</alwaysOn>
           <updateRate>60.0</updateRate>
@@ -31,6 +30,6 @@
           <imageTopicName>image_raw</imageTopicName>
           <cameraInfoTopicName>camera_info</cameraInfoTopicName>
-          <frameName>${link_name}</frameName>
-          <hackBaseline>0.0</hackBaseline>
+          <frameName>${name}</frameName>
+          <hackBaseline>0.07</hackBaseline>
           <distortionK1>0.0</distortionK1>
           <distortionK2>0.0</distortionK2>

File: model_description/urdf/sensor/camera.urdf.xacro (robot description, xacro)
@@ -1,28 +1,31 @@
 <?xml version="1.0"?>
 <robot xmlns:xacro="http://ros.org/wiki/xacro">
-  <xacro:include filename="$(find model_description)/urdf/common.xacro" />
-  <xacro:include filename="$[find model_description]/urdf/materials.xacro"/>
-  <xacro:macro name="camera_link_v0" params="parent_link link_name *joint_origin">
-	<joint name="${link_name}_joint" type="fixed">
-	  <insert_block name="*joint_origin"/>
-	  <parent link="${parent_link}"/>
-	  <child link="${link_name}"/>
+  <xacro:include filename="$(find model_description)/urdf/common.xacro"/>
+  <xacro:macro name="camera_link_v0" params="parent name *joint_origin">
+	<joint name="${name}_joint" type="fixed">
+	  <insert_block name="joint_origin"/>
+	  <parent link="${parent}"/>
+	  <child link="${name}"/>
 	</joint>
-	<link name="${link_name}">
+	<link name="${name}">
 	  <visual>
-		<magerial name="black"/>
+		<origin rpy="0 ${M_PI/2} 0"/>
+		<material name="black"/>
 		<geometry>
-		  <mesh filename="package://model_description/meshes/camera.stl"/>
+		  <mesh filename="package://model_description/meshes/camera.stl" scale="0.05 0.05 0.05"/>
 		</geometry>
 	  </visual>
 	  <collision>
+		<origin rpy="0 ${M_PI/2} 0"/>
 		<geometry>
-		  <mesh filename="package://model_description/meshes/camera.stl"/>
+		  <mesh filename="package://model_description/meshes/camera.stl" scale="0.05 0.05 0.05"/>
 		</geometry>
 	  </collision>
-	  <inertia>
+	  <inertial>
 		<mass value="0.07"/>
-		<inertia ixx="0.1" iyy="0.1" izz="0.1"/>
-	  </inertia>
+		<inertia ixx="0.001" ixy="0" ixz="0"
+				 iyy="0.001" iyz="0"
+				 izz="0.001" />
+	  </inertial>
 	</link>
   </xacro:macro>
